Commit message: little little changes

File: src/description/urdf/robot_base.xacro (robot description, xacro)
@@ -1,149 +1,139 @@
 <?xml version="1.0"?>
 <robot xmlns:xacro="http://www.ros.org/wiki/xacro">
-<xacro:macro name="base">
-  <xacro:property name="base_length" value="0.5"/>
-  <xacro:property name="base_width" value="0.4"/>
-  <xacro:property name="base_height" value="0.2"/>
-  <xacro:property name="wheel_radius" value="0.075"/>
-  <xacro:property name="wheel_width" value="0.04"/>
-  <xacro:property name="wheel_x_offset" value="0.18"/>
-  <xacro:property name="wheel_y_offset" value="0.22"/>
-<link name="base_footprint"/>
-<joint name="base_footprint_joint" type="fixed">
-  <parent link="base_footprint"/>
-  <child link="base_link"/>
-  <origin xyz="0 0 0" rpy="0 0 0"/>
-</joint>
-  <link name="base_link">
-    <visual>
-      <geometry>
-        <box size="${base_length} ${base_width} ${base_height}"/>
-      </geometry>
-      <origin xyz="0 0 ${base_height/2 + 0.05}"/>
-      <material name="body_color">
-        <color rgba="0.15 0.15 0.18 1"/>
-      </material>
-    </visual>
-    <collision>
-      <geometry>
-        <box size="${base_length} ${base_width} ${base_height}"/>
-      </geometry>
-      <origin xyz="0 0 ${base_height/2 + 0.05}"/>
-    </collision>
-    <inertial>
-      <mass value="10.0"/>
-      <origin xyz="0 0 ${base_height/2 + 0.05}"/>
-      <inertia
-        ixx="0.2"
-        iyy="0.2"
-        izz="0.2"
-        ixy="0" ixz="0" iyz="0"/>
-    </inertial>
-  </link>
-  <gazebo reference="base_link">
-    <self_collide>false</self_collide>
-  </gazebo>
-  <link name="imu_link">
-    <visual>
-      <geometry>
-        <box size="0.03 0.03 0.02"/>
-      </geometry>
-      <material name="orange">
-        <color rgba="1 0.5 0 1"/>
-      </material>
-      <origin xyz="0 0 0.15" rpy="0 0 0"/>
-    </visual>
-  </link>
-  <joint name="imu_joint" type="fixed">
-    <parent link="base_link"/>
-    <child link="imu_link"/>
-    <origin xyz="0 0 0.15"/>
-  </joint>
-  <link name="gps_link">
-    <visual>
-      <geometry>
-        <box size="0.03 0.03 0.02"/>
-      </geometry>
-      <material name="white">
-        <color rgba="1 1 1 1"/>
-      </material>
-      <origin xyz="0 0 0.2" rpy="0 0 0"/>
-    </visual>
-  </link>
-  <joint name="gps_joint" type="fixed">
-    <parent link="base_link"/>
-    <child link="gps_link"/>
-    <origin xyz="0 0 0.2"/>
-  </joint>
-  <link name="lidar_link">
-    <visual>
-      <geometry>
-        <cylinder radius="0.04" length="0.05"/>
-      </geometry>
-      <origin xyz="0.1 0 0.15" rpy="0 0 0"/>
-      <material name="gray">
-        <color rgba="0.6 0.6 0.6 1.0"/>
-      </material>
-    </visual>
-  </link>
-  <joint name="lidar_joint" type="fixed">
-    <parent link="base_link"/>
-    <child link="lidar_link"/>
-    <origin xyz="0.11 0 0.15"/>
-  </joint>
-  <link name="camera_link">
-    <origin xyz="0.15 0 0.12" rpy="0 0 0"/>
-  </link>
-  <joint name="camera_joint" type="fixed">
-    <parent link="base_link"/>
-    <child link="camera_link"/>
-    <origin xyz="0.15 0 0.12"/>
-  </joint>
-  <xacro:macro name="wheel" params="name x y">
-    <link name="${name}_link">
+  <xacro:macro name="base">
+    <xacro:property name="base_length" value="0.5"/>
+    <xacro:property name="base_width" value="0.4"/>
+    <xacro:property name="base_height" value="0.2"/>
+    <xacro:property name="wheel_radius" value="0.075"/>
+    <xacro:property name="wheel_width" value="0.04"/>
+    <xacro:property name="wheel_x_offset" value="0.18"/>
+    <xacro:property name="wheel_y_offset" value="0.22"/>
+    <link name="base_link">
       <visual>
-        <origin rpy="1.5708 0 0"/>
         <geometry>
-          <cylinder radius="${wheel_radius}" length="${wheel_width}"/>
+          <box size="${base_length} ${base_width} ${base_height}"/>
         </geometry>
-        <material name="black">
-          <color rgba="0.05 0.05 0.05 1"/>
+        <origin xyz="0 0 ${base_height/2}" rpy="0 0 0"/>
+        <material name="body_color">
+          <color rgba="0.15 0.15 0.18 1"/>
         </material>
       </visual>
       <collision>
-        <origin rpy="1.5708 0 0"/>
         <geometry>
-          <cylinder radius="${wheel_radius}" length="${wheel_width}"/>
+          <box size="${base_length} ${base_width} ${base_height}"/>
         </geometry>
+        <origin xyz="0 0 ${base_height/2}" rpy="0 0 0"/>
       </collision>
       <inertial>
-        <mass value="1.0"/>
-        <origin xyz="0 0 0"/>
-        <inertia
-          ixx="0.01"
-          iyy="0.01"
-          izz="0.005"
-          ixy="0" ixz="0" iyz="0"/>
+        <mass value="10.0"/>
+        <origin xyz="0 0 ${base_height/2}"/>
+        <inertia ixx="0.2" iyy="0.2" izz="0.2" ixy="0" ixz="0" iyz="0"/>
       </inertial>
     </link>
-    <joint name="${name}_joint" type="continuous">
+    <gazebo reference="base_link">
+      <self_collide>false</self_collide>
+    </gazebo>
+    <link name="imu_link">
+      <visual>
+        <geometry>
+          <box size="0.03 0.03 0.02"/>
+        </geometry>
+        <origin xyz="0 0 0"/>
+        <material name="orange">
+          <color rgba="1 0.5 0 1"/>
+        </material>
+      </visual>
+    </link>
+    <joint name="imu_joint" type="fixed">
       <parent link="base_link"/>
-      <child link="${name}_link"/>
-      <origin xyz="${x} ${y} ${wheel_radius}"/>
-      <axis xyz="0 1 0"/>
+      <child link="imu_link"/>
+      <origin xyz="0 0 0.15"/>
     </joint>
+    <link name="gps_link">
+      <visual>
+        <geometry>
+          <box size="0.03 0.03 0.02"/>
+        </geometry>
+        <origin xyz="0 0 0"/>
+        <material name="white">
+          <color rgba="1 1 1 1"/>
+        </material>
+      </visual>
+    </link>
+    <joint name="gps_joint" type="fixed">
+      <parent link="base_link"/>
+      <child link="gps_link"/>
+      <origin xyz="0 0 0.2"/>
+    </joint>
+    <link name="lidar_link">
+      <visual>
+        <geometry>
+          <cylinder radius="0.04" length="0.05"/>
+        </geometry>
+        <origin xyz="0 0 0"/>
+        <material name="gray">
+          <color rgba="0.6 0.6 0.6 1.0"/>
+        </material>
+      </visual>
+      <collision>
+        <geometry>
+          <cylinder radius="0.04" length="0.05"/>
+        </geometry>
+        <origin xyz="0 0 0"/>
+      </collision>
+    </link>
+    <joint name="lidar_joint" type="fixed">
+      <parent link="base_link"/>
+      <child link="lidar_link"/>
+      <origin xyz="0.11 0 0.22"/>
+    </joint>
+    <link name="camera_link"/>
+    <joint name="camera_joint" type="fixed">
+      <parent link="base_link"/>
+      <child link="camera_link"/>
+      <origin xyz="0.15 0 0.12"/>
+    </joint>
+    <xacro:macro name="wheel" params="name x y">
+      <link name="${name}_link">
+        <visual>
+          <origin rpy="1.5708 0 0"/>
+          <geometry>
+            <cylinder radius="${wheel_radius}" length="${wheel_width}"/>
+          </geometry>
+          <material name="black">
+            <color rgba="0.05 0.05 0.05 1"/>
+          </material>
+        </visual>
+        <collision>
+          <origin rpy="1.5708 0 0"/>
+          <geometry>
+            <cylinder radius="${wheel_radius}" length="${wheel_width}"/>
+          </geometry>
+        </collision>
+        <inertial>
+          <mass value="1.0"/>
+          <origin xyz="0 0 0"/>
+          <inertia ixx="0.01" iyy="0.01" izz="0.005" ixy="0" ixz="0" iyz="0"/>
+        </inertial>
+      </link>
+      <joint name="${name}_joint" type="continuous">
+        <parent link="base_link"/>
+        <child link="${name}_link"/>
+        <origin xyz="${x} ${y} ${wheel_radius}"/>
+        <axis xyz="0 1 0"/>
+      </joint>
+    </xacro:macro>
+    <xacro:wheel name="front_left_wheel"
+                 x="${wheel_x_offset}"
+                 y="${wheel_y_offset}"/>
+    <xacro:wheel name="rear_left_wheel"
+                 x="-${wheel_x_offset}"
+                 y="${wheel_y_offset}"/>
+    <xacro:wheel name="front_right_wheel"
+                 x="${wheel_x_offset}"
+                 y="-${wheel_y_offset}"/>
+    <xacro:wheel name="rear_right_wheel"
+                 x="-${wheel_x_offset}"
+                 y="-${wheel_y_offset}"/>
   </xacro:macro>
-  <xacro:wheel name="front_left_wheel"
-               x="${wheel_x_offset}"
-               y="${wheel_y_offset}"/>
-  <xacro:wheel name="rear_left_wheel"
-               x="-${wheel_x_offset}"
-               y="${wheel_y_offset}"/>
-  <xacro:wheel name="front_right_wheel"
-               x="${wheel_x_offset}"
-               y="-${wheel_y_offset}"/>
-  <xacro:wheel name="rear_right_wheel"
-               x="-${wheel_x_offset}"
-               y="-${wheel_y_offset}"/>
-</xacro:macro>
 </robot>

File: src/description/urdf/robot_sensors.xacro (robot description, xacro)
@@ -22,5 +22,5 @@
         <topic>/scan</topic>
         <visualize>true</visualize>
-        <frame_id>lidar_link</frame_id>
+        <gz_frame_id>lidar_link</gz_frame_id>
         <lidar>
           <scan>
